File: hardware/TinyViolin.sch (KiCad schematic (older format))
At the start: 47 parts, among them J1 AVR-ISP-6, J2 503182-1852, SW1 SW_SPDT, SW2 SW_Push, SW3 SW_Push, SW4 SW_Push, SW5 SW_Push, SW6 SW_Push, U1 ATmega328PB-AU, U2 TPS613222ADBVT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

Commit message: Updated symbol fields
Parts:
- removed SW2: SW_Push, symbol Switch:SW_Push
- added C6: 22uF, Capacitor_SMD:C_0805_2012Metric_Pad1.15x1.40mm_HandSolder, symbol Device:C
- added SW2: Tactile, SW_1825910-7, symbol 1825910-7:1825910-7
- C5: value 2.2uF -> 22uF
- J2: Field4 WM12834CT-ND -> (none); Field5 5031821852 -> (none); Field6 https://www.digikey.com/product-detail/en/molex/5031821852/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 -> (none); Field7 MICRO SD NORMAL ULTRALOWPRO8CKTE -> (none); Field8 Molex -> (none)
- L1: footprint (none) -> Inductor_SMD:L_1206_3216Metric_Pad1.42x1.75mm_HandSolder; Part Number (none) -> LQM31PN2R2M00L
- LS1: footprint (none) -> Connector_Wire:SolderWirePad_1x02_P3.81mm_Drill0.8mm; Part Number (none) -> SP-1605
- R1: footprint (none) -> Resistor_SMD:R_0805_2012Metric_Pad1.15x1.40mm_HandSolder; Part Number (none) -> RMCF0805FT1M00
- R2: value 5 -> 10k; footprint (none) -> Resistor_SMD:R_0805_2012Metric_Pad1.15x1.40mm_HandSolder; Part Number (none) -> RNCP0805FTD4R70
- R3: value 10k -> 5
- RV1: Part Number (none) -> PTA4543-2015DPB103
- SW1: Part Number (none) -> MFS101D-8-Z
- SW3, SW4, SW5, SW6: Part Number (none) -> D6L90 F2 LFS
- U2: Field4 Unavailable -> (none); Field5 TPS613222ADBVT -> (none); Field6 6-uA Quiescent Current, 1.8-A Switch Current Boost Converte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 -> (none); Field7 Texas Instruments -> (none); Field8 None -> (none)
- renumbered C9 to C10, C6 to C7, C7 to C8, C8 to C9
Connections:
- net +5V: now also C6.1
- net GND: now also C6.2, SW2.3, SW2.4
- net ~RST: now also SW2.1, SW2.2
Other:
- moved on the sheet: C8, C9, D2, J2, R4, TP3, TP4, TP5, TP6, TP7, TP8, U3
