File: hardware/TinyViolin.sch (KiCad schematic (older format))
At the start: 46 parts, among them J1 AVR-ISP-6, J2 503182-1852, SW1 SW_SPDT, SW2 Tactile, SW3 SW_Push, SW4 SW_Push, SW5 SW_Push, SW6 SW_Push, U1 ATmega328-PU, U2 TPS613222ADBVT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

Commit message: Fixed labels
Parts:
- J1: value AVR-ISP-6 -> ICSP
- U2: value TPS613222ADBVT -> BOOST
- U3: value MIC5504-3.3YM5 -> REG
Changed lines of the file:
@@
 Wire Wire Line
 	6400 6050 6400 6200
-Text Label 2300 6400 0    50   ~ 0
+Text Label 2300 4300 0    50   ~ 0
 SPEAKER
 Text Label 5650 5950 2    50   ~ 0
@@
 NoConn ~ 2300 6500
 NoConn ~ 2300 4200
-NoConn ~ 2300 4300
+NoConn ~ 2300 6400
 NoConn ~ 2300 5200
 NoConn ~ 2300 5300
@@
 P 4350 2400
 F 0 "U2" H 4350 3070 50  0000 C CNN
-F 1 "TPS613222ADBVT" H 4350 2979 50  0000 C CNN
+F 1 "BOOST" H 4350 2979 50  0000 C CNN
 F 2 "SOT95P280X145-5N" H 4350 2400 50  0001 L BNN
 F 3 "http://www.ti.com/lit/ds/symlink/tps61322.pdf" H 4350 2400 50  0001 L BNN
@@
 P 3400 3950
 F 0 "J1" H 3121 4046 50  0000 R CNN
-F 1 "AVR-ISP-6" H 3121 3955 50  0000 R CNN
+F 1 "ICSP" H 3121 3955 50  0000 R CNN
 F 2 "Connector_PinHeader_2.54mm:PinHeader_2x03_P2.54mm_Vertical" V 3150 4000 50  0001 C CNN
 F 3 "https://katalog.we-online.de/em/datasheet/6120xx21621.pdf" H 2125 3400 50  0001 C CNN
@@
 F 4 "ECE-A0JKS101	" H 6200 5950 50  0001 C CNN "Part Number"
 	1    6200 5950
-	0    1    1    0
+	0    -1   -1   0
 $EndComp
 $Comp
@@
 P 7200 2300
 F 0 "U3" H 7200 2667 50  0000 C CNN
-F 1 "MIC5504-3.3YM5" H 7200 2576 50  0000 C CNN
+F 1 "REG" H 7200 2576 50  0000 C CNN
 F 2 "Package_TO_SOT_SMD:SOT-23-5" H 7200 1900 50  0001 C CNN
 F 3 "http://ww1.microchip.com/downloads/en/DeviceDoc/MIC550X.pdf" H 6950 2550 50  0001 C CNN

Commit message: Wrote code for buttons and leds
Parts:
- U1: footprint Package_DIP:DIP-28_W7.62mm_Socket_LongPads -> Package_DIP:DIP-28_W7.62mm_LongPads
Changed lines of the file:
@@
 F 0 "U1" H 1300 3950 50  0000 R CNN
 F 1 "ATmega328-PU" H 2350 3950 50  0000 R CNN
-F 2 "Package_DIP:DIP-28_W7.62mm_Socket_LongPads" H 1700 5400 50  0001 C CIN
+F 2 "Package_DIP:DIP-28_W7.62mm_LongPads" H 1700 5400 50  0001 C CIN
 F 3 "http://ww1.microchip.com/downloads/en/DeviceDoc/ATmega328_P%20AVR%20MCU%20with%20picoPower%20Technology%20Data%20Sheet%2040001984A.pdf" H 1700 5400 50  0001 C CNN
 	1    1700 5400

Commit message: Updated pcb for manufacture
Parts:
- SW1: Part Number 1825255-1 -> MHS122
Changed lines of the file:
@@
 F 1 "SW_SPDT" H 2600 2694 50  0000 C CNN
 F 2 "MHS122:MHS122" H 2600 2500 50  0001 C CNN
-F 3 "https://www.te.com/commerce/DocumentDelivery/DDEController?Action=srchrtrv&DocNm=1825255&DocType=Customer+Drawing&DocLang=English" H 2600 2500 50  0001 C CNN
-F 4 "1825255-1" H 2600 2500 50  0001 C CNN "Part Number"
+F 3 "https://media.digikey.com/pdf/Data%20Sheets/APEM%20Components%20PDFs/MHS_Series.PDF" H 2600 2500 50  0001 C CNN
+F 4 "MHS122" H 2600 2500 50  0001 C CNN "Part Number"
 	1    2600 2500
 	1    0    0    -1

Commit message: Updated pcb with fixes
Parts:
- removed C7: 120pF, Capacitor_SMD:C_0805_2012Metric_Pad1.15x1.40mm_HandSolder, symbol Device:C
- removed C8, C9: 1uF, Capacitor_SMD:C_1206_3216Metric_Pad1.42x1.75mm_HandSolder, symbol Device:C
- removed D1: D_Schottky, DO219:DO219-AB, symbol Device:D_Schottky
- removed D3, D4, D5, D6: RGB_LED, LED_THT:LED_D5.0mm-4_RGB, symbol RGB_LED:RGB_LED
- removed R3: 5, Resistor_SMD:R_0805_2012Metric_Pad1.15x1.40mm_HandSolder, symbol Device:R
- removed TP4: 3.3V, TestPoint:TestPoint_Plated_Hole_D2.0mm, symbol Connector:TestPoint
- removed U3: REG, Package_TO_SOT_SMD:SOT-23-5, symbol Regulator_Linear:MIC5504-3.3YM5
- added D3, D4, D5, D6: LED, LED_THT:LED_D5.0mm, symbol Device:LED
- added R4, R5, R6, R7: 150, Resistor_SMD:R_0805_2012Metric_Pad1.15x1.40mm_HandSolder, symbol Device:R
- C4: value 2.2uF -> 22uF
- R3: renamed from R4; Part Number RMCF0805FT220R -> RNCP0805FTD150R
- SW3, SW4, SW5, SW6: footprint D6:D6 -> D6:TL1105; Part Number D6L90 F2 LFS -> TL1105BF160Q
- TP1, TP2: footprint TestPoint:TestPoint_Plated_Hole_D2.0mm -> TestPoint:TestPoint_Pad_D1.0mm
- TP3: value 5V -> V3.3; footprint TestPoint:TestPoint_Plated_Hole_D2.0mm -> TestPoint:TestPoint_Pad_D1.0mm
- U1: symbol MCU_Microchip_ATmega:ATmega328-PU -> TinyViolin-rescue:ATmega328-PU-MCU_Microchip_ATmega
- U2: Part Number TPS613222ADBVR -> TPS613221ADBVR
Connections:
- net labels added: LED1, LED2, LED3, LED4, VBOOST
- net labels removed: +5V, LEDS, SNUB, VSW
- wire segments 75 -> 49
- no-connect marks 25 -> 21
Other:
- moved on the sheet: BT1, C4, D2, L1, R3, SW1, TP1, TP2

Commit message: Connected 3.3V to SD card
Connections:
- net +3.3V is gone; now on net +3V3: J2.4 (VDD)
Changed lines of the file:
@@
 Text Label 9100 5000 2    50   ~ 0
 MISO
-Text Label 9100 4900 2    50   ~ 0
-GND
 Text Label 9100 4800 2    50   ~ 0
 SCK
-Text Label 9100 4700 2    50   ~ 0
-+3.3V
 Text Label 9100 4500 2    50   ~ 0
 SS
@@
 	9550 4400 9800 4400
 Wire Wire Line
-	9100 4700 9800 4700
-Wire Wire Line
-	9100 4900 9800 4900
-Wire Wire Line
 	9550 5100 9800 5100
 NoConn ~ 9800 5300
@@
 	3300 2600 3650 2600
 NoConn ~ 9800 5600
+$Comp
+L power:GND #PWR?
+U 1 1 5DCB43D5
+P 8750 4900
+F 0 "#PWR?" H 8750 4650 50  0001 C CNN
+F 1 "GND" H 8755 4727 50  0000 C CNN
+F 2 "" H 8750 4900 50  0001 C CNN
+F 3 "" H 8750 4900 50  0001 C CNN
+	1    8750 4900
+	1    0    0    -1
+$EndComp
+$Comp
+L power:+3.3V #PWR?
+U 1 1 5DCB4722
+P 8750 4700
+F 0 "#PWR?" H 8750 4550 50  0001 C CNN
+F 1 "+3.3V" H 8765 4873 50  0000 C CNN
+F 2 "" H 8750 4700 50  0001 C CNN
+F 3 "" H 8750 4700 50  0001 C CNN
+	1    8750 4700
+	1    0    0    -1
+$EndComp
+Wire Wire Line
+	8750 4700 9800 4700
+Wire Wire Line
+	8750 4900 9800 4900
 $EndSCHEMATC

Commit message: Prepared pcb for re-manufacturing
Parts:
- added C7: 100nF, Capacitor_SMD:C_0805_2012Metric_Pad1.15x1.40mm_HandSolder, symbol Device:C
- J1: Part Number 61200621621 -> (none)
- R2: Part Number RNCP0805FTD4R70 -> RNCP0805FTD10K0
- R3: Part Number RNCP0805FTD150R -> RMCF0805FT220R
- R4, R5, R6, R7: value 150 -> 220
Connections:
- net +3V3: now also R3.1, C7.1; no longer D2.2 (A)
- net GND: now also D2.1 (K), C7.2; no longer R3.2
- new net: D2.2 (A), R3.2
Other:
- moved on the sheet: D2, R3
Changed lines of the file:
@@
 EESchema Schematic File Version 4
 LIBS:TinyViolin-cache
-EELAYER 30 0
+EELAYER 26 0
 EELAYER END
 $Descr A4 11693 8268
@@
 L Device:R R3
 U 1 1 5DABDF08
-P 6250 2650
-F 0 "R3" H 6320 2696 50  0000 L CNN
-F 1 "220" H 6320 2605 50  0000 L CNN
-F 2 "Resistor_SMD:R_0805_2012Metric_Pad1.15x1.40mm_HandSolder" V 6180 2650 50  0001 C CNN
-F 3 "https://www.seielect.com/catalog/sei-rmcf_rmcp.pdf" H 6250 2650 50  0001 C CNN
-F 4 "RNCP0805FTD150R" H 6250 2650 50  0001 C CNN "Part Number"
-	1    6250 2650
+P 6250 2300
+F 0 "R3" H 6320 2346 50  0000 L CNN
+F 1 "220" H 6320 2255 50  0000 L CNN
+F 2 "Resistor_SMD:R_0805_2012Metric_Pad1.15x1.40mm_HandSolder" V 6180 2300 50  0001 C CNN
+F 3 "https://www.seielect.com/catalog/sei-rmcf_rmcp.pdf" H 6250 2300 50  0001 C CNN
+F 4 "RMCF0805FT220R" H 6250 2300 50  0001 C CNN "Part Number"
+	1    6250 2300
 	1    0    0    -1
 $EndComp
@@
 L Device:LED D2
 U 1 1 5DABCDE0
-P 6250 2300
-F 0 "D2" V 6289 2183 50  0000 R CNN
-F 1 "LED" V 6198 2183 50  0000 R CNN
-F 2 "LED_SMD:LED_0805_2012Metric_Pad1.15x1.40mm_HandSolder" H 6250 2300 50  0001 C CNN
-F 3 "https://dammedia.osram.info/media/resource/hires/osram-dam-2493936/LG%20R971.pdf" H 6250 2300 50  0001 C CNN
-F 4 "LG R971-KN-1	" H 6250 2300 50  0001 C CNN "Part Number"
-	1    6250 2300
+P 6250 2650
+F 0 "D2" V 6289 2533 50  0000 R CNN
+F 1 "LED" V 6198 2533 50  0000 R CNN
+F 2 "LED_SMD:LED_0805_2012Metric_Pad1.15x1.40mm_HandSolder" H 6250 2650 50  0001 C CNN
+F 3 "https://dammedia.osram.info/media/resource/hires/osram-dam-2493936/LG%20R971.pdf" H 6250 2650 50  0001 C CNN
+F 4 "LG R971-KN-1	" H 6250 2650 50  0001 C CNN "Part Number"
+	1    6250 2650
 	0    -1   -1   0
 $EndComp
@@
 F 1 "ICSP" H 3121 3955 50  0000 R CNN
 F 2 "Connector_PinHeader_2.54mm:PinHeader_2x03_P2.54mm_Vertical" V 3150 4000 50  0001 C CNN
-F 3 "https://katalog.we-online.de/em/datasheet/6120xx21621.pdf" H 2125 3400 50  0001 C CNN
-F 4 "61200621621" H 3400 3950 50  0001 C CNN "Part Number"
+F 3 "~" H 2125 3400 50  0001 C CNN
+F 4 "~" H 3400 3950 50  0001 C CNN "Part Number"
 	1    3400 3950
 	1    0    0    -1
@@
 F 2 "Resistor_SMD:R_0805_2012Metric_Pad1.15x1.40mm_HandSolder" V 3280 5900 50  0001 C CNN
 F 3 "https://www.seielect.com/catalog/sei-rncp.pdf" H 3350 5900 50  0001 C CNN
-F 4 "RNCP0805FTD4R70" H 3350 5900 50  0001 C CNN "Part Number"
+F 4 "RNCP0805FTD10K0" H 3350 5900 50  0001 C CNN "Part Number"
 	1    3350 5900
 	1    0    0    -1
@@
 P 4850 4800
 F 0 "R4" H 4920 4846 50  0000 L CNN
-F 1 "150" H 4920 4755 50  0000 L CNN
+F 1 "220" H 4920 4755 50  0000 L CNN
 F 2 "Resistor_SMD:R_0805_2012Metric_Pad1.15x1.40mm_HandSolder" V 4780 4800 50  0001 C CNN
 F 3 "https://www.seielect.com/catalog/sei-rmcf_rmcp.pdf" H 4850 4800 50  0001 C CNN
@@
 P 5850 4800
 F 0 "R5" H 5920 4846 50  0000 L CNN
-F 1 "150" H 5920 4755 50  0000 L CNN
+F 1 "220" H 5920 4755 50  0000 L CNN
 F 2 "Resistor_SMD:R_0805_2012Metric_Pad1.15x1.40mm_HandSolder" V 5780 4800 50  0001 C CNN
 F 3 "https://www.seielect.com/catalog/sei-rmcf_rmcp.pdf" H 5850 4800 50  0001 C CNN
@@
 P 6850 4800
 F 0 "R6" H 6920 4846 50  0000 L CNN
-F 1 "150" H 6920 4755 50  0000 L CNN
+F 1 "220" H 6920 4755 50  0000 L CNN
 F 2 "Resistor_SMD:R_0805_2012Metric_Pad1.15x1.40mm_HandSolder" V 6780 4800 50  0001 C CNN
 F 3 "https://www.seielect.com/catalog/sei-rmcf_rmcp.pdf" H 6850 4800 50  0001 C CNN
@@
 P 7850 4800
 F 0 "R7" H 7920 4846 50  0000 L CNN
-F 1 "150" H 7920 4755 50  0000 L CNN
+F 1 "220" H 7920 4755 50  0000 L CNN
 F 2 "Resistor_SMD:R_0805_2012Metric_Pad1.15x1.40mm_HandSolder" V 7780 4800 50  0001 C CNN
 F 3 "https://www.seielect.com/catalog/sei-rmcf_rmcp.pdf" H 7850 4800 50  0001 C CNN
@@
 NoConn ~ 9800 5600
 $Comp
-L power:GND #PWR?
+L power:GND #PWR0125
 U 1 1 5DCB43D5
-P 8750 4900
-F 0 "#PWR?" H 8750 4650 50  0001 C CNN
-F 1 "GND" H 8755 4727 50  0000 C CNN
-F 2 "" H 8750 4900 50  0001 C CNN
-F 3 "" H 8750 4900 50  0001 C CNN
-	1    8750 4900
-	1    0    0    -1
-$EndComp
-$Comp
-L power:+3.3V #PWR?
+P 8450 4950
+F 0 "#PWR0125" H 8450 4700 50  0001 C CNN
+F 1 "GND" H 8455 4777 50  0000 C CNN
+F 2 "" H 8450 4950 50  0001 C CNN
+F 3 "" H 8450 4950 50  0001 C CNN
+	1    8450 4950
+	1    0    0    -1
+$EndComp
+$Comp
+L power:+3.3V #PWR0126
 U 1 1 5DCB4722
-P 8750 4700
-F 0 "#PWR?" H 8750 4550 50  0001 C CNN
-F 1 "+3.3V" H 8765 4873 50  0000 C CNN
-F 2 "" H 8750 4700 50  0001 C CNN
-F 3 "" H 8750 4700 50  0001 C CNN
-	1    8750 4700
+P 8450 4650
+F 0 "#PWR0126" H 8450 4500 50  0001 C CNN
+F 1 "+3.3V" H 8465 4823 50  0000 C CNN
+F 2 "" H 8450 4650 50  0001 C CNN
+F 3 "" H 8450 4650 50  0001 C CNN
+	1    8450 4650
 	1    0    0    -1
 $EndComp
@@
 Wire Wire Line
 	8750 4900 9800 4900
+$Comp
+L Device:C C7
+U 1 1 5DCC2B84
+P 8450 4800
+F 0 "C7" H 8565 4846 50  0000 L CNN
+F 1 "100nF" H 8565 4755 50  0000 L CNN
+F 2 "Capacitor_SMD:C_0805_2012Metric_Pad1.15x1.40mm_HandSolder" H 8488 4650 50  0001 C CNN
+F 3 "http://www.samsungsem.com/kr/support/product-search/mlcc/CL21B104JBCNNNC.jsp" H 8450 4800 50  0001 C CNN
+F 4 "CL21B104JBCNNNC" H 8450 4800 50  0001 C CNN "Part Number"
+	1    8450 4800
+	1    0    0    -1
+$EndComp
+Wire Wire Line
+	8750 4700 8750 4650
+Wire Wire Line
+	8750 4650 8450 4650
+Connection ~ 8450 4650
+Wire Wire Line
+	8450 4950 8750 4950
+Wire Wire Line
+	8750 4950 8750 4900
+Connection ~ 8450 4950
 $EndSCHEMATC

Commit message: Got main thing working
Connections:
- net +3V3: now also J1.2 (VCC)
Changed lines of the file:
@@
 L power:+3.3V #PWR0130
 U 1 1 5DA9A983
-P 3150 3450
-F 0 "#PWR0130" H 3150 3300 50  0001 C CNN
-F 1 "+3.3V" H 3165 3623 50  0000 C CNN
-F 2 "" H 3150 3450 50  0001 C CNN
-F 3 "" H 3150 3450 50  0001 C CNN
-	1    3150 3450
+P 3300 3450
+F 0 "#PWR0130" H 3300 3300 50  0001 C CNN
+F 1 "+3.3V" H 3315 3623 50  0000 C CNN
+F 2 "" H 3300 3450 50  0001 C CNN
+F 3 "" H 3300 3450 50  0001 C CNN
+	1    3300 3450
 	1    0    0    -1
 $EndComp

Commit message: Changed battery on PCB
Parts:
- removed BT1: BAT-HLD-001-THM, LINX_BAT-HLD-001-THM, symbol BAT-HLD-001-THM:BAT-HLD-001-THM
- removed U1: ATmega328-PU, Package_DIP:DIP-28_W7.62mm_LongPads, symbol TinyViolin-rescue:ATmega328-PU-MCU_Microchip_ATmega
- added BT1: BCAAAPC, BAT_BCAAAPC, symbol BCAAAPC:BCAAAPC
- added U1: ATmega328-PU, Package_DIP:DIP-28_W7.62mm_LongPads, symbol MCU_Microchip_ATmega:ATmega328-PU
- Y1: value Crystal 16MHz -> Crystal 8MHz; Part Number ABL-16.000MHZ-B2 -> ABL-8.000MHZ-B2
Connections:
- wire segments 53 -> 52
Other:
- moved on the sheet: SW1, TP1, TP2
Changed lines of the file:
@@
 NoConn ~ 3650 2400
 NoConn ~ 3650 2200
-NoConn ~ 2650 2400
+NoConn ~ 2250 2500
 Text Label 3800 4050 0    50   ~ 0
 ~RST
@@
 L power:GND #PWR0121
 U 1 1 5DAA4917
-P 1450 2900
-F 0 "#PWR0121" H 1450 2650 50  0001 C CNN
-F 1 "GND" H 1455 2727 50  0000 C CNN
-F 2 "" H 1450 2900 50  0001 C CNN
-F 3 "" H 1450 2900 50  0001 C CNN
-	1    1450 2900
+P 1450 3200
+F 0 "#PWR0121" H 1450 2950 50  0001 C CNN
+F 1 "GND" H 1455 3027 50  0000 C CNN
+F 2 "" H 1450 3200 50  0001 C CNN
+F 3 "" H 1450 3200 50  0001 C CNN
+	1    1450 3200
 	1    0    0    -1
 $EndComp
@@
 NoConn ~ 2300 5600
 Wire Wire Line
-	1450 2900 1100 2900
+	1450 3200 1100 3200
 $Comp
 L power:+3.3V #PWR0130
@@
 L Switch:SW_SPDT SW1
 U 1 1 5DAA50F5
-P 2450 2500
-F 0 "SW1" H 2450 2785 50  0000 C CNN
-F 1 "SW_SPDT" H 2450 2694 50  0000 C CNN
-F 2 "MHS122:MHS122" H 2450 2500 50  0001 C CNN
-F 3 "https://media.digikey.com/pdf/Data%20Sheets/APEM%20Components%20PDFs/MHS_Series.PDF" H 2450 2500 50  0001 C CNN
-F 4 "MHS122" H 2450 2500 50  0001 C CNN "Part Number"
-	1    2450 2500
-	1    0    0    -1
+P 2450 2600
+F 0 "SW1" H 2450 2885 50  0000 C CNN
+F 1 "SW_SPDT" H 2450 2794 50  0000 C CNN
+F 2 "MHS122:MHS122" H 2450 2600 50  0001 C CNN
+F 3 "https://media.digikey.com/pdf/Data%20Sheets/APEM%20Components%20PDFs/MHS_Series.PDF" H 2450 2600 50  0001 C CNN
+F 4 "MHS122" H 2450 2600 50  0001 C CNN "Part Number"
+	1    2450 2600
+	-1   0    0    1
 $EndComp
 $Comp
@@
 P 3000 4850
 F 0 "Y1" V 3046 4719 50  0000 R CNN
-F 1 "Crystal 16MHz" V 2955 4719 50  0000 R CNN
+F 1 "Crystal 8MHz" V 2955 4719 50  0000 R CNN
 F 2 "Crystal:Crystal_HC49-U_Vertical" H 3000 4850 50  0001 C CNN
 F 3 "https://abracon.com/Resonators/ABL.pdf" H 3000 4850 50  0001 C CNN
-F 4 "ABL-16.000MHZ-B2	" H 3000 4850 50  0001 C CNN "Part Number"
+F 4 "ABL-8.000MHZ-B2" H 3000 4850 50  0001 C CNN "Part Number"
 	1    3000 4850
 	0    -1   -1   0
@@
 L Connector:TestPoint TP1
 U 1 1 5DB550E0
-P 1450 2500
-F 0 "TP1" H 1508 2618 50  0000 L CNN
-F 1 "VBT" H 1508 2527 50  0000 L CNN
-F 2 "TestPoint:TestPoint_Pad_D1.0mm" H 1650 2500 50  0001 C CNN
-F 3 "~" H 1650 2500 50  0001 C CNN
-F 4 "~" H 1450 2500 50  0001 C CNN "Part Number"
-	1    1450 2500
+P 1450 2700
+F 0 "TP1" H 1508 2818 50  0000 L CNN
+F 1 "VBT" H 1508 2727 50  0000 L CNN
+F 2 "TestPoint:TestPoint_Pad_D1.0mm" H 1650 2700 50  0001 C CNN
+F 3 "~" H 1650 2700 50  0001 C CNN
+F 4 "~" H 1450 2700 50  0001 C CNN "Part Number"
+	1    1450 2700
 	1    0    0    -1
 $EndComp
@@
 L Connector:TestPoint TP2
 U 1 1 5DB55599
-P 1100 2500
-F 0 "TP2" H 1158 2618 50  0000 L CNN
-F 1 "GND" H 1158 2527 50  0000 L CNN
-F 2 "TestPoint:TestPoint_Pad_D1.0mm" H 1300 2500 50  0001 C CNN
-F 3 "~" H 1300 2500 50  0001 C CNN
-F 4 "~" H 1100 2500 50  0001 C CNN "Part Number"
-	1    1100 2500
+P 1100 2700
+F 0 "TP2" H 1158 2818 50  0000 L CNN
+F 1 "GND" H 1158 2727 50  0000 L CNN
+F 2 "TestPoint:TestPoint_Pad_D1.0mm" H 1300 2700 50  0001 C CNN
+F 3 "~" H 1300 2700 50  0001 C CNN
+F 4 "~" H 1100 2700 50  0001 C CNN "Part Number"
+	1    1100 2700
 	1    0    0    -1
 $EndComp
@@
 Connection ~ 4450 6250
 $Comp
-L BAT-HLD-001-THM:BAT-HLD-001-THM BT1
-U 1 1 5DB41DC7
-P 1450 2700
-F 0 "BT1" V 1496 2567 50  0000 R CNN
-F 1 "BAT-HLD-001-THM" V 1405 2567 50  0000 R CNN
-F 2 "LINX_BAT-HLD-001-THM" H 1450 2700 50  0001 L BNN
-F 3 "https://linxtechnologies.com/wp/wp-content/uploads/bat-hld-001-thm.pdf" H 1450 2700 50  0001 L BNN
-F 4 "BAT-HLD-001-THM" H -250 1100 50  0001 C CNN "Part Number"
-	1    1450 2700
-	0    -1   -1   0
-$EndComp
-Wire Wire Line
-	1700 3900 1800 3900
-Connection ~ 1700 3900
-$Comp
-L TinyViolin-rescue:ATmega328-PU-MCU_Microchip_ATmega U1
-U 1 1 5DB4AE2D
-P 1700 5400
-F 0 "U1" H 1300 3950 50  0000 R CNN
-F 1 "ATmega328-PU" H 2350 3950 50  0000 R CNN
-F 2 "Package_DIP:DIP-28_W7.62mm_LongPads" H 1700 5400 50  0001 C CIN
-F 3 "http://ww1.microchip.com/downloads/en/DeviceDoc/ATmega328_P%20AVR%20MCU%20with%20picoPower%20Technology%20Data%20Sheet%2040001984A.pdf" H 1700 5400 50  0001 C CNN
-	1    1700 5400
-	1    0    0    -1
-$EndComp
-$Comp
 L Connector:Conn_01x01_Male H1
 U 1 1 5DB4E674
@@
 NoConn ~ 3650 6850
 NoConn ~ 3650 7100
-Connection ~ 1450 2900
-Wire Wire Line
-	1100 2500 1100 2900
-Wire Wire Line
-	2250 2500 1450 2500
-Connection ~ 1450 2500
+Wire Wire Line
+	2250 2700 1450 2700
 Wire Wire Line
 	9100 4600 9800 4600
@@
 Wire Wire Line
 	4850 5650 4850 5800
-Text Label 1750 2500 0    50   ~ 0
+Text Label 1750 2700 0    50   ~ 0
 BAT
 Text Label 2700 2600 0    50   ~ 0
@@
 	8750 4950 8750 4900
 Connection ~ 8450 4950
+$Comp
+L BCAAAPC:BCAAAPC BT1
+U 1 1 5DD563D0
+P 1450 3000
+F 0 "BT1" V 1354 3130 50  0000 L CNN
+F 1 "BCAAAPC" V 1445 3130 50  0000 L CNN
+F 2 "BAT_BCAAAPC" H 1450 3000 50  0001 L BNN
+F 3 "http://www.memoryprotectiondevices.com/datasheets/BCAAAPC-datasheet.pdf" H 1450 3000 50  0001 L BNN
+F 4 "BCAAAPC" H 1450 3000 50  0001 L BNN "Part Number"
+	1    1450 3000
+	0    1    1    0
+$EndComp
+Wire Wire Line
+	1100 2700 1100 3200
+Connection ~ 1450 2700
+Connection ~ 1450 3200
+$Comp
+L MCU_Microchip_ATmega:ATmega328-PU U1
+U 1 1 5DD59E82
+P 1700 5400
+F 0 "U1" H 1900 3950 50  0000 R CNN
+F 1 "ATmega328-PU" H 2400 3850 50  0000 R CNN
+F 2 "Package_DIP:DIP-28_W7.62mm_LongPads" H 1700 5400 50  0001 C CIN
+F 3 "http://ww1.microchip.com/downloads/en/DeviceDoc/ATmega328_P%20AVR%20MCU%20with%20picoPower%20Technology%20Data%20Sheet%2040001984A.pdf" H 1700 5400 50  0001 C CNN
+	1    1700 5400
+	1    0    0    -1
+$EndComp
 $EndSCHEMATC
