File: hardware/TinyViolin.kicad_pcb (KiCad board)
At the start: 2 copper layers, 100 x 80 mm, 46 parts, among them J1 ICSP, J2 503182-1852, SW1 SW_SPDT, SW2 Tactile, SW3 SW_Push, SW4 SW_Push, SW5 SW_Push, SW6 SW_Push, U1 ATmega328-PU, U2 BOOST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

Commit message: Updated pcb for manufacture
Parts:
- R3: value 5 -> 4.7
- moved H3 1.00 mm to (36.0, 94.0)
- moved H6 1.00 mm to (114.0, 94.0)
Changed lines of the file:
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@@
   )
   (module MountingHole:MountingHole_3.2mm_M3 (layer F.Cu)
-    (at 36 95)
+    (at 36 94)
     (descr "Mounting Hole 3.2mm, no annular, M3")
     (tags "mounting hole 3.2mm no annular m3")
@@
   )
   (module MountingHole:MountingHole_3.2mm_M3 (layer F.Cu)
-    (at 114 95)
+    (at 114 94)
     (descr "Mounting Hole 3.2mm, no annular, M3")
     (tags "mounting hole 3.2mm no annular m3")
@@
       (effects (font (size 1 1) (thickness 0.15)))
     )
-    (fp_text value 5 (at -3 3 180) (layer F.SilkS)
+    (fp_text value 4.7 (at -3 3 180) (layer F.SilkS)
       (effects (font (size 1 1) (thickness 0.15)))
     )
@@
   (segment (start 27.54 54.54) (end 29.5 52.58) (width 0.25) (layer B.Cu) (net 1))
   (segment (start 29.5 52.58) (end 29.5 50.5) (width 0.25) (layer B.Cu) (net 1))
+  (segment (start 58.1 50.365) (end 58.1 50) (width 0.25) (layer B.Cu) (net 3))
   (segment (start 62.02 69.72) (end 60.3 68) (width 0.25) (layer B.Cu) (net 4))
   (segment (start 62.02 70.12) (end 62.02 69.72) (width 0.25) (layer B.Cu) (net 4))
@@
   (segment (start 22.5 52.04) (end 25 54.54) (width 0.25) (layer B.Cu) (net 6))
   (segment (start 22.5 50) (end 22.5 52.04) (width 0.25) (layer B.Cu) (net 6))
-  (segment (start 58.1 50.365) (end 58.1 50) (width 0.25) (layer B.Cu) (net 3))
   (segment (start 57.1 50.365) (end 57.1 50) (width 0.25) (layer B.Cu) (net 7))
   (segment (start 59.235 52.5) (end 57.1 50.365) (width 0.25) (layer B.Cu) (net 7))

Commit message: Updated pcb with fixes
Parts:
- removed C7: 120pF, Capacitor_SMD:C_0805_2012Metric_Pad1.15x1.40mm_HandSolder
- removed C8, C9: 1uF, Capacitor_SMD:C_1206_3216Metric_Pad1.42x1.75mm_HandSolder
- removed D1: D_Schottky, DO219:DO219-AB
- removed the R3 at (113.5, 79.5)
- removed TP4: 3.3V, TestPoint:TestPoint_Plated_Hole_D2.0mm
- removed U3: REG, Package_TO_SOT_SMD:SOT-23-5
- added R4: 150, Resistor_SMD:R_0805_2012Metric_Pad1.15x1.40mm_HandSolder, F.Cu at (64.0, 51.0)
- added R5: 150, Resistor_SMD:R_0805_2012Metric_Pad1.15x1.40mm_HandSolder, F.Cu at (79.0, 51.0)
- added R6: 150, Resistor_SMD:R_0805_2012Metric_Pad1.15x1.40mm_HandSolder, F.Cu at (94.0, 51.0)
- added R7: 150, Resistor_SMD:R_0805_2012Metric_Pad1.15x1.40mm_HandSolder, F.Cu at (109.0, 51.0)
- BT1: footprint LINX_BAT-HLD-001-THM -> BAT-HLD-001-THM:LINX_BAT-HLD-001-THM
- C4: value 2.2uF -> 22uF
- D3, D4, D5, D6: value RGB_LED -> LED; footprint LED_THT:LED_D5.0mm-4_RGB -> LED_THT:LED_D5.0mm
- J2: footprint MOLEX_503182-1852 -> 503182-1852:MOLEX_503182-1852
- SW2: footprint SW_1825910-7 -> 1825910-7:SW_1825910-7
- SW3, SW4, SW5, SW6: footprint D6:D6 -> D6:TL1105
- TP1, TP2: footprint TestPoint:TestPoint_Plated_Hole_D2.0mm -> TestPoint:TestPoint_Pad_D1.0mm
- TP3: value 5V -> V3.3; footprint TestPoint:TestPoint_Plated_Hole_D2.0mm -> TestPoint:TestPoint_Pad_D1.0mm
- U2: footprint SOT95P280X145-5N -> TPS613222ADBVT:SOT95P280X145-5N
- moved TP3 53.1 mm to (110.0, 60.0)
- moved TP2 39.6 mm to (50.0, 95.0)
- moved TP1 12.0 mm to (101.5, 87.5)
- moved D2 8.06 mm to (56.5, 97.5), turned to 180 degrees
- moved R2 8.00 mm to (55.5, 91.0)
- moved SW2 8.00 mm to (62.0, 92.0)
- moved L1 6.02 mm to (114.0, 77.0), turned to 90 degrees
- moved BT1 5.00 mm to (80.0, 90.0)
- moved SW3 3.54 mm to (59.0, 26.0), turned to 0 degrees
- moved SW4 3.54 mm to (74.0, 26.0), turned to 0 degrees
- moved SW5 3.54 mm to (89.0, 26.0), turned to 0 degrees
- moved SW6 3.54 mm to (104.0, 26.0), turned to 0 degrees
- moved J1 3.00 mm to (25.0, 49.0)
- moved R3 2.55 mm to (61.0, 97.5), turned to 0 degrees
- moved J2 2.00 mm to (30.0, 38.0), turned to 270 degrees
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- renumbered R4 to R3
Connections:
- net /VSW renamed /VBOOST
- C5 pad 1: +5V -> +3V3
- C6 pad 1: +5V -> +3V3
- D3 pad 1: /LEDS -> GND
- D3 pad 2: +5V -> Net-(D3-Pad2)
- D4 pad 1: Net-(D3-Pad4) -> GND
- D4 pad 2: +5V -> Net-(D4-Pad2)
- D5 pad 1: Net-(D4-Pad4) -> GND
- D5 pad 2: +5V -> Net-(D5-Pad2)
- D6 pad 1: Net-(D5-Pad4) -> GND
- D6 pad 2: +5V -> Net-(D6-Pad2)
- H1 pad 1: Net-(H1-Pad1) -> (no net)
- H2 pad 1: Net-(H2-Pad1) -> (no net)
- H3 pad 1: Net-(H3-Pad1) -> (no net)
- H4 pad 1: Net-(H4-Pad1) -> (no net)
- H5 pad 1: Net-(H5-Pad1) -> (no net)
- H6 pad 1: Net-(H6-Pad1) -> (no net)
- J1 pad 2: +3V3 -> (no net)
- J2 pad 1: Net-(J2-Pad1) -> (no net)
- J2 pad 4: /+3.3V -> (no net)
- J2 pad 8: Net-(J2-Pad8) -> (no net)
- J2 pad DT: Net-(J2-PadDT) -> (no net)
- J2 pad SW: Net-(J2-PadSW) -> (no net)
- SW1 pad 1: Net-(SW1-Pad1) -> (no net)
- TP3 pad 1: +5V -> +3V3
- U1 pad 11: Net-(U1-Pad11) -> /LED2
- U1 pad 12: Net-(U1-Pad12) -> /PB1
- U1 pad 13: Net-(U1-Pad13) -> /LED1
- U1 pad 14: Net-(U1-Pad14) -> (no net)
- U1 pad 2: /PB4 -> /LED4
- U1 pad 21: Net-(U1-Pad21) -> (no net)
- U1 pad 24: Net-(U1-Pad24) -> (no net)
- U1 pad 25: Net-(U1-Pad25) -> (no net)
- U1 pad 26: Net-(U1-Pad26) -> (no net)
- U1 pad 27: Net-(U1-Pad27) -> (no net)
- U1 pad 28: Net-(U1-Pad28) -> (no net)
- U1 pad 3: /PB3 -> /LED3
- U1 pad 4: /PB2 -> /PB4
- U1 pad 5: /PB1 -> /PB3
- U1 pad 6: /LEDS -> /PB2
- U2 pad 3: Net-(U2-Pad3) -> (no net)
- U2 pad 4: +5V -> +3V3
- U2 pad 5: Net-(U2-Pad5) -> (no net)
Routing:
- net /BAT: track 0.00 -> 43.1 mm
- net /BAT1: track 0.00 -> 30.8 mm
- net /LEDS: track 28.9 -> 0.00 mm
- net /LED4: track 0.00 -> 23.6 mm
- net /SS: track 46.6 -> 68.6 mm
- net GND: track 30.5 -> 50.5 mm, vias 7 -> 6
- net /SCK: track 94.2 -> 75.8 mm
- net /LED2: track 0.00 -> 17.7 mm
- net /LED3: track 0.00 -> 13.2 mm
- net /MISO: track 76.1 -> 64.1 mm
- net /LED1: track 0.00 -> 11.3 mm
- net Net-(D5-Pad4): track 11.2 -> 0.00 mm
- net Net-(D4-Pad4): track 11.2 -> 0.00 mm
- net Net-(D3-Pad4): track 11.2 -> 0.00 mm
- net /MOSI: track 69.6 -> 75.3 mm
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- removed copper zone on F.Cu, net +5V
- removed copper zone on F.Cu, net /BAT
- removed copper zone on F.Cu, net /BAT1
- removed copper zone on F.Cu, net /SNUB
- removed copper zone on F.Cu, net /VBOOST
- removed copper zone on F.Cu, net GND
Other:
- board text added: "Tiny Violin MM v1.1"
- board text removed: "+"
- board text removed: "-"
- board text removed: "."
- board text removed: "Tiny Violin MM v1.0"

Commit message: Fixed labels
Parts:
- renumbered TP1 to TPe

Commit message: Connected 3.3V to SD card
Parts:
- renumbered TPe to TP1
Connections:
- J2 pad 4: (no net) -> +3V3
Routing:
- net +3V3: track 0.00 -> 1.90 mm, vias 0 -> 1
Changed lines of the file:
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@@
     (thickness 1.6)
     (drawings 5)
-    (tracks 178)
+    (tracks 181)
     (zones 0)
     (modules 43)
@@
     (add_net GND)
   )
-  (module TPS613222ADBVT:SOT95P280X145-5N (layer F.Cu)
-    (at 115 70)
-    (attr smd)
-    (fp_text reference U2 (at 1.956 -3.289) (layer F.SilkS) hide
-      (effects (font (size 1.4 1.4) (thickness 0.05)))
-    )
-    (fp_text value BOOST (at 0 3.311) (layer F.SilkS)
-      (effects (font (size 1 1) (thickness 0.15)))
-    )
-    (fp_line (start 1.775 2.11) (end -1.775 2.11) (layer Eco1.User) (width 0.05))
-    (fp_line (start 1.775 -2.11) (end 1.775 2.11) (layer Eco1.User) (width 0.05))
-    (fp_line (start -1.775 -2.11) (end 1.775 -2.11) (layer Eco1.User) (width 0.05))
-    (fp_line (start -1.775 2.11) (end -1.775 -2.11) (layer Eco1.User) (width 0.05))
-    (fp_line (start 1.525 -0.875) (end 1.525 0.875) (layer Eco2.User) (width 0.127))
-    (fp_line (start -1.525 0.875) (end -1.525 -0.875) (layer Eco2.User) (width 0.127))
-    (fp_line (start -1.525 -0.875) (end 1.525 -0.875) (layer Eco2.User) (width 0.127))
-    (fp_line (start 1.525 0.875) (end -1.525 0.875) (layer Eco2.User) (width 0.127))
-    (fp_line (start 1.525 -0.33) (end 1.525 0.33) (layer F.SilkS) (width 0.127))
-    (fp_line (start -0.335 -0.875) (end 0.335 -0.875) (layer F.SilkS) (width 0.127))
-    (fp_line (start -1.525 0.33) (end -1.525 -0.33) (layer F.SilkS) (width 0.127))
-    (fp_circle (center -0.95 2.31) (end -0.85 2.31) (layer Eco2.User) (width 0.2))
-    (fp_circle (center -0.95 2.31) (end -0.85 2.31) (layer F.SilkS) (width 0.2))
-    (pad 5 smd rect (at -0.95 -1.255 180) (size 0.59 1.21) (layers F.Cu F.Paste F.Mask))
-    (pad 4 smd rect (at 0.95 -1.255 180) (size 0.59 1.21) (layers F.Cu F.Paste F.Mask)
-      (net 2 +3V3))
-    (pad 3 smd rect (at 0.95 1.255) (size 0.59 1.21) (layers F.Cu F.Paste F.Mask))
-    (pad 2 smd rect (at 0 1.255) (size 0.59 1.21) (layers F.Cu F.Paste F.Mask)
-      (net 9 GND))
-    (pad 1 smd rect (at -0.95 1.255) (size 0.59 1.21) (layers F.Cu F.Paste F.Mask)
-      (net 29 /VBOOST))
-  )
   (module 1825910-7:SW_1825910-7 (layer F.Cu)
     (at 62 92)
-    (fp_text reference SW2 (at -0.96119 -4.14014) (layer F.SilkS) hide
+    (fp_text reference SW2 (at -0.96119 -4.14014) (layer F.SilkS)
       (effects (font (size 1.00124 1.00124) (thickness 0.05)))
     )
-    (fp_text value Tactile (at -0.325215 4.11758) (layer F.SilkS) hide
+    (fp_text value Tactile (at -0.325215 4.11758) (layer F.SilkS)
       (effects (font (size 1.00062 1.00062) (thickness 0.05)))
     )
@@
     (at 30 38 270)
     (attr smd)
-    (fp_text reference J2 (at -8.64903 -4.21685 180) (layer B.SilkS) hide
+    (fp_text reference J2 (at -8.64903 -4.21685 180) (layer B.SilkS)
       (effects (font (size 1.00162 1.00162) (thickness 0.05)) (justify mirror))
     )
-    (fp_text value 503182-1852 (at 8.63712 -3.58418 180) (layer B.SilkS) hide
+    (fp_text value 503182-1852 (at 8.63712 -3.58418 180) (layer B.SilkS)
       (effects (font (size 1.00257 1.00257) (thickness 0.05)) (justify mirror))
     )
@@
     (pad 5 smd rect (at 1.5 6.355 270) (size 0.8 1.24) (layers B.Cu B.Paste B.Mask)
       (net 5 /SCK))
-    (pad 4 smd rect (at 0.4 6.355 270) (size 0.8 1.24) (layers B.Cu B.Paste B.Mask))
+    (pad 4 smd rect (at 0.4 6.355 270) (size 0.8 1.24) (layers B.Cu B.Paste B.Mask)
+      (net 2 +3V3))
     (pad 3 smd rect (at -0.7 6.355 270) (size 0.8 1.24) (layers B.Cu B.Paste B.Mask)
       (net 1 /MOSI))
@@
       (net 3 /SS))
     (pad 1 smd rect (at -2.9 6.355 270) (size 0.8 1.24) (layers B.Cu B.Paste B.Mask))
+  )
+  (module TPS613222ADBVT:SOT95P280X145-5N (layer F.Cu)
+    (at 115 70)
+    (attr smd)
+    (fp_text reference U2 (at 1.956 -3.289) (layer F.SilkS) hide
+      (effects (font (size 1.4 1.4) (thickness 0.05)))
+    )
+    (fp_text value BOOST (at 0 3.311) (layer F.SilkS)
+      (effects (font (size 1 1) (thickness 0.15)))
+    )
+    (fp_line (start 1.775 2.11) (end -1.775 2.11) (layer Eco1.User) (width 0.05))
+    (fp_line (start 1.775 -2.11) (end 1.775 2.11) (layer Eco1.User) (width 0.05))
+    (fp_line (start -1.775 -2.11) (end 1.775 -2.11) (layer Eco1.User) (width 0.05))
+    (fp_line (start -1.775 2.11) (end -1.775 -2.11) (layer Eco1.User) (width 0.05))
+    (fp_line (start 1.525 -0.875) (end 1.525 0.875) (layer Eco2.User) (width 0.127))
+    (fp_line (start -1.525 0.875) (end -1.525 -0.875) (layer Eco2.User) (width 0.127))
+    (fp_line (start -1.525 -0.875) (end 1.525 -0.875) (layer Eco2.User) (width 0.127))
+    (fp_line (start 1.525 0.875) (end -1.525 0.875) (layer Eco2.User) (width 0.127))
+    (fp_line (start 1.525 -0.33) (end 1.525 0.33) (layer F.SilkS) (width 0.127))
+    (fp_line (start -0.335 -0.875) (end 0.335 -0.875) (layer F.SilkS) (width 0.127))
+    (fp_line (start -1.525 0.33) (end -1.525 -0.33) (layer F.SilkS) (width 0.127))
+    (fp_circle (center -0.95 2.31) (end -0.85 2.31) (layer Eco2.User) (width 0.2))
+    (fp_circle (center -0.95 2.31) (end -0.85 2.31) (layer F.SilkS) (width 0.2))
+    (pad 5 smd rect (at -0.95 -1.255 180) (size 0.59 1.21) (layers F.Cu F.Paste F.Mask))
+    (pad 4 smd rect (at 0.95 -1.255 180) (size 0.59 1.21) (layers F.Cu F.Paste F.Mask)
+      (net 2 +3V3))
+    (pad 3 smd rect (at 0.95 1.255) (size 0.59 1.21) (layers F.Cu F.Paste F.Mask))
+    (pad 2 smd rect (at 0 1.255) (size 0.59 1.21) (layers F.Cu F.Paste F.Mask)
+      (net 9 GND))
+    (pad 1 smd rect (at -0.95 1.255) (size 0.59 1.21) (layers F.Cu F.Paste F.Mask)
+      (net 29 /VBOOST))
   )
   (module BAT-HLD-001-THM:LINX_BAT-HLD-001-THM (layer B.Cu)
@@
     (tags "test point SMD pad")
     (attr virtual)
-    (fp_text reference TPe (at 0 -1.448) (layer F.SilkS) hide
+    (fp_text reference TP1 (at 0 -1.448) (layer F.SilkS) hide
       (effects (font (size 1 1) (thickness 0.15)))
     )
@@
   (segment (start 27.54 64.96) (end 27.5 65) (width 0.5) (layer F.Cu) (net 9))
   (segment (start 27.54 54.08) (end 27.54 64.96) (width 0.5) (layer F.Cu) (net 9))
+  (via (at 25.5 38.5) (size 0.8) (drill 0.4) (layers F.Cu B.Cu) (net 2))
+  (segment (start 25.4 38.4) (end 25.5 38.5) (width 0.5) (layer B.Cu) (net 2))
+  (segment (start 23.645 38.4) (end 25.4 38.4) (width 0.5) (layer B.Cu) (net 2))
   (segment (start 57.525 97.5) (end 59.975 97.5) (width 0.25) (layer F.Cu) (net 10))
   (segment (start 93.55 62.5) (end 94.5 63.45) (width 0.25) (layer B.Cu) (net 11))
